File: KiCad/GR_Varta_To_CR2032.sch (KiCad schematic (older format))
At the start: 4 parts, among them J1 S8401-46, J2 Conn_01x01, J3 Conn_01x01

Commit message: Add files via upload
Parts:
- D1: value 1N5819 -> 1N5711
Changed lines of the file:
@@
 P 5350 4450
 F 0 "D1" H 5350 4350 50  0000 C CNN
-F 1 "1N5819" H 5350 4550 50  0000 C CNN
+F 1 "1N5711" H 5350 4550 50  0000 C CNN
 F 2 "Diode_THT:D_DO-41_SOD81_P10.16mm_Horizontal" H 5350 4275 50  0001 C CNN
 F 3 "http://www.vishay.com/docs/88525/1n5817.pdf" H 5350 4450 50  0001 C CNN
